Commit message: joint1 영점을 180° 옮김 — 홈이 -172° 에서 +8° 로
형상은 하나도 안 바뀐다. 관절값을 읽는 기준만 바뀐다.

  URDF   joint1 origin rpy  [0 0 0] → [0 0 π]
  관절값  q_new = q_old − 180°  (mod 360)
  홈      joint1 -172.00° → +8.00°   나머지 4축은 그대로

왜
  홈의 joint1 이 -172° 라 리밋(±178)까지 6° 뿐이었다. 더 나쁜 것은 못 쓰는
  4° 구간이 **팔이 정면(툴 방위 0°)을 향하는 자리**였다는 점이다 — 작업
  방향 한복판이 막혀 있었다.

    전   홈 -172   좌/우 여유    6° / 350°   막힌 곳 = 정면
    후   홈   +8   좌/우 여유  186° / 170°   막힌 곳 = 뒤(차체)

  뒤쪽은 어차피 차체와 부딪히는 자리라 잃을 것이 없다.
  새 규약에서는 툴 방위 = joint1 이라 읽기도 쉬워진다.

수식 — 자식 pose = T_origin · Rot(axis, q) 이므로
  T_origin_new = T_origin_old · Rot(axis, offset)  →  q_new = q_old − offset
도구는 scripts/16_rotate_joint_zero.py 로 남겼다. 기구 담당이 새 URDF 를
주면 그 파일은 옛 영점이라 매번 돌려야 한다.

검증
  arm_v1·arm_v2 모두 홈에서 tool_frame·camera_mount·link5·jaw_l/r 의 world
  pose 를 옛 모델과 대조 — 위치차 0.0000mm / 자세차 0.0000°
  도달 반경 0.2~472.0mm, 최대 높이 428.1mm 그대로
  서버 기동 joint1=+8.0, EE (0.1596,0.0224,0.2908) — 옛 홈과 동일
  테스트 131개 통과

★★ 실물·Isaac 도 같이 맞춰야 한다. 안 맞추면 첫 지령에 팔이 반 바퀴 돈다.
  (A) joint1 서보의 기계 영점을 180° 옮기거나
  (B) 드라이버에서 지령·피드백 양쪽에 -180° 오프셋
  handoff/68 §3, handoff/69 §6, board 에 적었다.

파생물 재생성: _ik.urdf · body_with_arm_v2*.urdf · arms.json
꾸러미 두 개(for_echo_v4 / for_isaac)도 새 URDF·문서로 다시 말았다.
echo_v4 패치는 이제 05_teleop_sim.py 도 충돌한다(argparse 블록, 덩어리 1개).
어디를 어떻게 푸는지 04_적용방법.txt 에 적었다.

Co-Authored-By: Claude Opus 5 (1M context) <noreply@anthropic.com>

File: assets/arm_v1/arm_v1.urdf (robot description, URDF)
Before this commit: robot arm_new, 12 links, 11 joints
Joints:
- joint joint1: origin xyz=0 0 0.05505 rpy=0 0 0 -> xyz=0 0 0.05505 rpy=0 -0 3.14159265359

File: assets/arm_v1/arm_v1_ik.urdf (robot description, URDF)
Before this commit: robot arm_new_ik, 12 links, 11 joints
Joints:
- joint joint1: origin xyz=0 0 0.05505 rpy=0 0 0 -> xyz=0 0 0.05505 rpy=0 -0 3.14159265359

File: assets/arm_v1/arm_v1_nomimic.urdf (robot description, URDF)
Before this commit: robot arm_new_nomimic, 12 links, 11 joints
Joints:
- joint joint1: origin xyz=0 0 0.05505 rpy=0 0 0 -> xyz=0 0 0.05505 rpy=0 -0 3.14159265359

File: assets/arm_v2/arm_v2.urdf (robot description, URDF)
Before this commit: robot arm_new, 12 links, 11 joints
Joints:
- joint joint1: origin xyz=0 0 0.05505 rpy=0 0 0 -> xyz=0 0 0.05505 rpy=0 -0 3.14159265359

File: assets/arm_v2/arm_v2_ik.urdf (robot description, URDF)
Before this commit: robot arm_new2_ik, 12 links, 11 joints
Joints:
- joint joint1: origin xyz=0 0 0.05505 rpy=0 0 0 -> xyz=0 0 0.05505 rpy=0 -0 3.14159265359

File: assets/arm_v2/arm_v2_nomimic.urdf (robot description, URDF)
Before this commit: robot arm_new_nomimic, 12 links, 11 joints
Joints:
- joint joint1: origin xyz=0 0 0.05505 rpy=0 0 0 -> xyz=0 0 0.05505 rpy=0 -0 3.14159265359

File: assets/body/body_with_arm_v2.urdf (robot description, URDF)
Before this commit: robot body_with_arm_v2, 15 links, 14 joints
Joints:
- joint joint1: origin xyz=0 0 0.05505 rpy=0 0 0 -> xyz=0 0 0.05505 rpy=0 -0 3.14159265359

File: assets/body/body_with_arm_v2_nomimic.urdf (robot description, URDF)
Before this commit: robot body_with_arm_v2_nomimic, 15 links, 14 joints
Joints:
- joint joint1: origin xyz=0 0 0.05505 rpy=0 0 0 -> xyz=0 0 0.05505 rpy=0 -0 3.14159265359

Commit message: 기구 담당 회신(71) 반영 — 개구 82.52 · joint1 원복 · 그리퍼 180° 재체결 모델 · 회신 72
전달본 robotarm_delivery_2026-09-03 을 대조했다. 메시 10개·_props 는 동일하고
URDF 는 그리퍼 리밋(gripper_joint -15.30~47.50°, rocker_r -54.57~7.93°)과
mimic 계수만 바뀌었다. 스윕은 56점(10~120°) → 95점(10~198°).

개구 57 → 82.52 mm
  57 은 기계 한계가 아니라 스윕 범위였다. 캔(66)·페트병 몸통(65)·종이컵(80)
  전부 잡힌다. 하드웨어 변경 없음. 로드맵의 "제약 2" 는 해소.

★ 전달본 gripper_map.py 의 7차 다항식이 발산한다
  최고차항이 -0.0 으로 찍혀(반올림) 서보 100° 부터 틀리고 198° 에서 개구
  -1092 mm, 로커L 1639°. 그래서 다항식을 버리고 실측 95점을 보간표로 쓰는
  판을 scripts/17_fit_gripper_map.py 로 만들어 교체했다. 원본은
  gripper_map_delivered_2026-09-03.py 로 보관.
  검산: 기구 담당 서보각 표와 2° 안, 198° 관절값이 URDF 리밋과 0.1° 안.
  gripper_link 는 신판 joint_rad() 를 쓰고 개구 최대를 OPENING_RANGE_MM 에서 읽는다.
  트리거 0/0.5/1 → 개구 82.5/41.5/0.5 mm, 조 원점 간격 107.7/66.7/25.7 mm 확인.

★ joint1 영점 이동(8bba238)은 되돌렸다 — 전제가 틀렸다
  joint1 은 팔 전체를 통째로 돌려서 카메라·툴 상대 관계를 못 바꾼다. 카메라
  위/아래는 j5 가 정한다. 사용자 자세가 j1=-172 로 간 진짜 이유는 카메라
  (link5 +x)를 위로 두려면 팔꿈치를 뒤 분지로 접고 j1 을 반 바퀴 돌려야
  했기 때문이다. 관절값 규약은 원래대로.

  대신 기구 담당 제안대로 "그리퍼 조립체를 motor5 장착면에서 180° 돌려
  체결"(볼트원 4×90°, 부품 0개)을 joint5 origin rpy [0 0 -π] 로 모델했다.
  motor5 엔코더 영점은 그대로라 캘리브레이션 오프셋이 없다.
  홈 [0, -54.51, +84.45, +80.78, +4.90]° — 거울 분지. 사용자 VR 자세와 세계
  형상 동일(정면 8° 요만 다름): tool·camera·link5·jaw 위치차 0.02mm/0.005°.
  툴 (161.2,0,290.8) · 아래 20.7° · 카메라 위 32.7mm · j1 여유 ±178°.

joint5 리밋 ±178 → ±90° (config). 케이블 꼬임 경고(67 §7-2) 반영, 72 §4-5.

문서: ARM_VERSIONS(09-03 항목) · 68 §2.3/§3 · 69 §6/§7 · docs/07 · 아티팩트 ·
board · 꾸러미 3개 재구성. handoff/72_MECH_REPLY2.txt 로 질문 7개에 답했고
쓰레기통은 정면이 C920 을 가리므로 측면을 권했다(광선 기하 계산 첨부).
71 회신 원본은 handoff/ 에 보관.

검증: 테스트 131개 통과 · 서버 기동 joint1=0 · dof_mismatch None.

Co-Authored-By: Claude Fable 5.1 <noreply@anthropic.com>

File: assets/arm_v1/arm_v1.urdf (robot description, URDF)
Before this commit: robot arm_new, 12 links, 11 joints
Joints:
- joint joint1: origin xyz=0 0 0.05505 rpy=0 -0 3.14159265359 -> xyz=0 0 0.05505 rpy=0 0 0
- joint joint5: origin xyz=0 0 0 rpy=0 0 0 -> xyz=0 0 0 rpy=0 -0 -3.14159265359

File: assets/arm_v1/arm_v1_ik.urdf (robot description, URDF)
Before this commit: robot arm_new, 12 links, 11 joints
Joints:
- joint joint1: origin xyz=0 0 0.05505 rpy=0 -0 3.14159265359 -> xyz=0 0 0.05505 rpy=0 0 0
- joint joint5: origin xyz=0 0 0 rpy=0 0 0 -> xyz=0 0 0 rpy=0 -0 -3.14159265359

File: assets/arm_v1/arm_v1_nomimic.urdf (robot description, URDF)
Before this commit: robot arm_new_nomimic, 12 links, 11 joints
Joints:
- joint joint1: origin xyz=0 0 0.05505 rpy=0 -0 3.14159265359 -> xyz=0 0 0.05505 rpy=0 0 0
- joint joint5: origin xyz=0 0 0 rpy=0 0 0 -> xyz=0 0 0 rpy=0 -0 -3.14159265359

File: assets/arm_v2/arm_v2.urdf (robot description, URDF)
Before this commit: robot arm_new, 12 links, 11 joints
Joints:
- joint gripper_joint: limit lower=-0.267032722 upper=0.590295874 effort=1.5 velocity=3 -> lower=-0.267032722 upper=0.828992955 effort=1.5 velocity=3
- joint jaw_l_joint: limit lower=-0.957328596 upper=0.957328596 effort=1.5 velocity=3 -> lower=-1.19602568 upper=1.19602568 effort=1.5 velocity=3
- joint jaw_r_joint: limit lower=-0.758756397 upper=0.758756397 effort=1.5 velocity=3 -> lower=-1.19079361 upper=1.19079361 effort=1.5 velocity=3
- joint joint1: origin xyz=0 0 0.05505 rpy=0 -0 3.14159265359 -> xyz=0 0 0.05505 rpy=0 0 0
- joint joint5: origin xyz=0 0 0 rpy=0 0 0 -> xyz=0 0 0 rpy=0 -0 -3.14159265359
- joint rocker_r_joint: limit lower=-0.520385894 upper=0.138370504 effort=1.5 velocity=3 -> lower=-0.952423108 upper=0.138370504 effort=1.5 velocity=3; mimic joint=gripper_joint multiplier=-0.731853091 offset=-0.0257247368 -> joint=gripper_joint multiplier=-0.960999949 offset=-0.0278370813

File: assets/arm_v2/arm_v2_ik.urdf (robot description, URDF)
Before this commit: robot arm_new, 12 links, 11 joints
Joints:
- joint joint1: origin xyz=0 0 0.05505 rpy=0 -0 3.14159265359 -> xyz=0 0 0.05505 rpy=0 0 0
- joint joint5: origin xyz=0 0 0 rpy=0 0 0 -> xyz=0 0 0 rpy=0 -0 -3.14159265359

File: assets/arm_v2/arm_v2_nomimic.urdf (robot description, URDF)
Before this commit: robot arm_new_nomimic, 12 links, 11 joints
Joints:
- joint gripper_joint: limit lower=-0.267032722 upper=0.590295874 effort=1.5 velocity=3 -> lower=-0.267032722 upper=0.828992955 effort=1.5 velocity=3
- joint jaw_l_joint: limit lower=-0.957328596 upper=0.957328596 effort=1.5 velocity=3 -> lower=-1.19602568 upper=1.19602568 effort=1.5 velocity=3
- joint jaw_r_joint: limit lower=-0.758756397 upper=0.758756397 effort=1.5 velocity=3 -> lower=-1.19079361 upper=1.19079361 effort=1.5 velocity=3
- joint joint1: origin xyz=0 0 0.05505 rpy=0 -0 3.14159265359 -> xyz=0 0 0.05505 rpy=0 0 0
- joint joint5: origin xyz=0 0 0 rpy=0 0 0 -> xyz=0 0 0 rpy=0 -0 -3.14159265359
- joint rocker_r_joint: limit lower=-0.520385894 upper=0.138370504 effort=1.5 velocity=3 -> lower=-0.952423108 upper=0.138370504 effort=1.5 velocity=3

File: assets/body/body_with_arm_v2.urdf (robot description, URDF)
Before this commit: robot body_with_arm_v2, 15 links, 14 joints
Joints:
- joint gripper_joint: limit lower=-0.267032722 upper=0.590295874 effort=1.5 velocity=3 -> lower=-0.267032722 upper=0.828992955 effort=1.5 velocity=3
- joint jaw_l_joint: limit lower=-0.957328596 upper=0.957328596 effort=1.5 velocity=3 -> lower=-1.19602568 upper=1.19602568 effort=1.5 velocity=3
- joint jaw_r_joint: limit lower=-0.758756397 upper=0.758756397 effort=1.5 velocity=3 -> lower=-1.19079361 upper=1.19079361 effort=1.5 velocity=3
- joint joint1: origin xyz=0 0 0.05505 rpy=0 -0 3.14159265359 -> xyz=0 0 0.05505 rpy=0 0 0
- joint joint5: origin xyz=0 0 0 rpy=0 0 0 -> xyz=0 0 0 rpy=0 -0 -3.14159265359
- joint rocker_r_joint: limit lower=-0.520385894 upper=0.138370504 effort=1.5 velocity=3 -> lower=-0.952423108 upper=0.138370504 effort=1.5 velocity=3; mimic joint=gripper_joint multiplier=-0.731853091 offset=-0.0257247368 -> joint=gripper_joint multiplier=-0.960999949 offset=-0.0278370813

File: assets/body/body_with_arm_v2_nomimic.urdf (robot description, URDF)
Before this commit: robot body_with_arm_v2_nomimic, 15 links, 14 joints
Joints:
- joint gripper_joint: limit lower=-0.267032722 upper=0.590295874 effort=1.5 velocity=3 -> lower=-0.267032722 upper=0.828992955 effort=1.5 velocity=3
- joint jaw_l_joint: limit lower=-0.957328596 upper=0.957328596 effort=1.5 velocity=3 -> lower=-1.19602568 upper=1.19602568 effort=1.5 velocity=3
- joint jaw_r_joint: limit lower=-0.758756397 upper=0.758756397 effort=1.5 velocity=3 -> lower=-1.19079361 upper=1.19079361 effort=1.5 velocity=3
- joint joint1: origin xyz=0 0 0.05505 rpy=0 -0 3.14159265359 -> xyz=0 0 0.05505 rpy=0 0 0
- joint joint5: origin xyz=0 0 0 rpy=0 0 0 -> xyz=0 0 0 rpy=0 -0 -3.14159265359
- joint rocker_r_joint: limit lower=-0.520385894 upper=0.138370504 effort=1.5 velocity=3 -> lower=-0.952423108 upper=0.138370504 effort=1.5 velocity=3
